Commit message: with controller

File: urdf/rr_bot_urdf.urdf (robot description, URDF)
Before this commit: robot rr_bot_urdf, 3 links, 2 joints
Links:
- added link world
Joints:
- added joint base_joint: type fixed, parent world, child base_link, origin xyz=0.0 0.0 0.17 rpy=0 0 0
- joint joint_1: origin xyz=0 0 0.15 rpy=3.1416 -1.5708 0 -> xyz=0 0 0.15 rpy=3.1416 -1.5708 3.1416
